Commit message: add some plugin sensor in URDF robot

File: my_robot_description/urdf/macros.xacro (robot description, xacro)
@@ -25,5 +25,5 @@
         </visual>
     </xacro:macro>
-    <xacro:macro name="wheel" params="name radius width *origin">
+    <xacro:macro name="wheel" params="name *origin">
         <link name="wheel_${name}_link">
             <inertial>
@@ -35,5 +35,5 @@
                 <origin xyz="0.0 0.0 0.0" rpy="${PI/2} 0.0 0.0"/>
                 <geometry>
-                    <cylinder radius="${radius}" length="${width}"/>
+                    <cylinder radius="${wheel_radius}" length="${wheel_width}"/>
                 </geometry>
                 <material name="black"/>
@@ -42,5 +42,5 @@
                 <origin xyz="0.0 0.0 0.0" rpy="${PI/2} 0.0 0.0"/>
                 <geometry>
-                    <cylinder radius="${radius}" length="${width}"/>
+                    <cylinder radius="${wheel_radius}" length="${wheel_width}"/>
                 </geometry>
             </collision>
@@ -52,5 +52,5 @@
             <xacro:insert_block name="origin"/>
         </joint>
-        <xacro:gazebo_wheel name="${name}"/>
+        <xacro:wheel_transmission name="${name}"/>
     </xacro:macro>
 </robot>

File: my_robot_description/urdf/my_robot.gazebo.xacro (robot description, xacro)
@@ -1,20 +1,149 @@
 <?xml version="1.0"?>
 <robot name="my_robot" xmlns:xacro="http://www.ros.org/wiki/xacro">
+    <gazebo reference="base_link">
+        <material>Gazebo/SkyBlue</material>
+	    <turnGravityOff>false</turnGravityOff>
+    </gazebo>
+    <gazebo reference="base_scan">
+        <material>Gazebo/Grey</material>
+	    <turnGravityOff>false</turnGravityOff>
+    </gazebo>
+    <xacro:macro name="wheel_transmission" params="name">
+        <gazebo reference="wheel_${name}_link">
+            <mu1 value="1.0"/>
+            <mu2 value="1.0"/>
+            <kp value="10000000.0"/>
+            <kd value="1.0"/>
+            <fdir1 value="0.2"/>
+            <material>Gazebo/Black</material>
+	        <turnGravityOff>false</turnGravityOff>
+        </gazebo>
+        <!-- <transmission name="wheel_${name}_trans">
+  		    <type>transmission_interface/SimpleTransmission</type>
+  		    <actuator name="wheel_${name}_motor">
+                <hardwareInterface>hardware_interface/VelocityJointInterface</hardwareInterface>
+			    <mechanicalReduction>1</mechanicalReduction>
+  		    </actuator>
+  		    <joint name="wheel_${name}_joint">
+			    <hardwareInterface>hardware_interface/VelocityJointInterface</hardwareInterface>
+  		    </joint>
+        </transmission> -->
+    </xacro:macro>
+    <xacro:if value="${use_gazebo_simulation}">
+        <gazebo>
+            <plugin name="differential_drive_controller" filename="libgazebo_ros_diff_drive.so">
+                <alwaysOn>true</alwaysOn>
+                <legacyMode>false</legacyMode>
+                <updateRate>100</updateRate>
+                <leftJoint>wheel_front_left_joint</leftJoint>
+                <rightJoint>wheel_front_right_joint</rightJoint>
+                <wheelSeparation>${wheel_separation}</wheelSeparation>
+                <wheelDiameter>${wheel_radius * 2}</wheelDiameter>
+                <wheelTorque>5</wheelTorque>
+                <torque>5</torque>
+                <commandTopic>/my_robot/cmd_vel</commandTopic>
+                <odometryTopic>odom</odometryTopic>
+                <odometryFrame>odom</odometryFrame>
+                <odometrySource >encoder</odometrySource >
+                <publishOdomTF>false</publishOdomTF>
+                <publishWheelTF>false</publishWheelTF>
+                <publishWheelJointState>false</publishWheelJointState>
+                <publishTf>1</publishTf>
+                <robotBaseFrame>base_footprint</robotBaseFrame>
+                <wheelAcceleration>0</wheelAcceleration>
+                <rosDebugLevel>na</rosDebugLevel>
+            </plugin>
+        </gazebo>
+        <gazebo>
+            <plugin name="differential_drive_controller" filename="libgazebo_ros_diff_drive.so">
+                <alwaysOn>true</alwaysOn>
+                <legacyMode>false</legacyMode>
+                <updateRate>100</updateRate>
+                <leftJoint>wheel_rear_left_joint</leftJoint>
+                <rightJoint>wheel_rear_right_joint</rightJoint>
+                <wheelSeparation>${wheel_separation}</wheelSeparation>
+                <wheelDiameter>${wheel_radius * 2}</wheelDiameter>
+                <wheelTorque>5</wheelTorque>
+                <torque>5</torque>
+                <commandTopic>/my_robot/cmd_vel</commandTopic>
+                <odometryTopic>odom</odometryTopic>
+                <odometryFrame>odom</odometryFrame>
+                <odometrySource >encoder</odometrySource >
+                <publishOdomTF>false</publishOdomTF>
+                <publishWheelTF>false</publishWheelTF>
+                <publishWheelJointState>false</publishWheelJointState>
+                <publishTf>1</publishTf>
+                <robotBaseFrame>base_footprint</robotBaseFrame>
+                <wheelAcceleration>0</wheelAcceleration>
+                <rosDebugLevel>na</rosDebugLevel>
+            </plugin>
+        </gazebo>
+        <gazebo reference="base_scan">
+            <sensor type="gpu_ray" name="lidar">
+                <pose>0 0 0 0 0 0</pose>
+                <visualize>true</visualize>
+                <update_rate>50</update_rate>
+                <ray>
+                    <scan>
+                        <horizontal>
+                        <samples>2000</samples>
+                        <resolution>1</resolution>
+                        <min_angle>-${PI}</min_angle>
+                        <max_angle>${PI}</max_angle>
+                        </horizontal>
+                    </scan>
+                    <range>
+                        <min>0.15</min>
+                        <max>10.0</max>
+                        <resolution>0.01</resolution>
+                    </range>
+                    <noise>
+                        <type>gaussian</type>
+                        <mean>0.0</mean>
+                        <stddev>0.01</stddev>
+                    </noise>
+                </ray>
+                <plugin name="gazebo_ros_head_hokuyo_controller" filename="libgazebo_ros_gpu_laser.so">
+                    <topicName>/my_robot/scan</topicName>
+                    <frameName>base_scan</frameName>
+                </plugin>
+            </sensor>
+        </gazebo>
+        <gazebo>
+            <plugin name="imu_plugin" filename="libgazebo_ros_imu.so">
+                <alwaysOn>true</alwaysOn>
+                <updateRate>50</updateRate>
+                <bodyName>imu_link</bodyName>
+                <frameName>imu_link</frameName>
+                <topicName>imu</topicName>
+                <serviceName>imu_service</serviceName>
+                <gaussianNoise>0.0</gaussianNoise>
+                <imu>
+                    <noise>
+                        <type>gaussian</type>
+                        <rate>
+                        <mean>0.0</mean>
+                        <stddev>2e-4</stddev>
+                        <bias_mean>0.0000075</bias_mean>
+                        <bias_stddev>0.0000008</bias_stddev>
+                        </rate>
+                        <accel>
+                        <mean>0.0</mean>
+                        <stddev>1.7e-2</stddev>
+                        <bias_mean>0.1</bias_mean>
+                        <bias_stddev>0.001</bias_stddev>
+                        </accel>
+                    </noise>
+                </imu>
+            </plugin>
+        </gazebo>
+    </xacro:if>
     <gazebo>
         <plugin name="gazebo_ros_control" filename="libgazebo_ros_control.so">
-            <robotNamespace>my_robot</robotNamespace>
+            <robotNamespace>/my_robot</robotNamespace>
+            <controlPeriod>0.001</controlPeriod>
+            <robotSimType>gazebo_ros_control/DefaultRobotHWSim</robotSimType>
             <legacyModeNS>true</legacyModeNS>
         </plugin>
     </gazebo>
-    <gazebo reference="base_link">
-        <material>Gazebo/SkyBlue</material>
-    </gazebo>
-    <gazebo reference="base_scan">
-        <material>Gazebo/Grey</material>
-    </gazebo>
-    <xacro:macro name="gazebo_wheel" params="name">
-        <gazebo reference="wheel_${name}_link">
-            <material>Gazebo/Black</material>
-        </gazebo>
-    </xacro:macro>
 </robot>

File: my_robot_description/urdf/my_robot.urdf.xacro (robot description, xacro)
@@ -9,4 +9,5 @@
     <xacro:property name="wheel_width" value="0.04"/>
     <xacro:property name="wheel_mass" value="0.4"/>
+    <xacro:property name="wheel_separation" value="0.33"/>
     <xacro:property name="support_length" value="0.03"/>
     <xacro:property name="support_width" value="0.03"/>
@@ -15,4 +16,5 @@
     <xacro:property name="top_width" value="0.26"/>
     <xacro:property name="top_height" value="0.005"/>
+    <xacro:property name="use_gazebo_simulation" value="${True}"/>
     <xacro:include filename="$(find my_robot_description)/urdf/macros.xacro"/>
     <xacro:include filename="$(find my_robot_description)/urdf/materials.xacro"/>
@@ -64,14 +66,14 @@
     <!-- End Chassis -->
     <!-- Wheel -->
-    <xacro:wheel name="front_left" radius="${wheel_radius}" width="${wheel_width}">
+    <xacro:wheel name="front_left">
         <origin xyz="0.1225 0.165 ${body_height/2}" rpy="0 0 0"/>
     </xacro:wheel>
-    <xacro:wheel name="rear_left" radius="${wheel_radius}" width="${wheel_width}">
+    <xacro:wheel name="rear_left">
         <origin xyz="-0.1225 0.165  ${body_height/2}" rpy="0 0 0"/>
     </xacro:wheel>
-    <xacro:wheel name="front_right" radius="${wheel_radius}" width="${wheel_width}">
+    <xacro:wheel name="front_right">
         <origin xyz="0.1225 -0.165 ${body_height/2}" rpy="0 0 0"/>
     </xacro:wheel>
-    <xacro:wheel name="rear_right" radius="${wheel_radius}" width="${wheel_width}">
+    <xacro:wheel name="rear_right">
         <origin xyz="-0.1225 -0.165 ${body_height/2}" rpy="0 0 0"/>
     </xacro:wheel>
@@ -104,3 +106,10 @@
     </joint>
     <!-- End Lidar -->
+    <!-- Imu -->
+    <link name="imu_link"/>
+    <joint name="imu_joint" type="fixed">
+        <parent link="base_link"/>
+        <child link="imu_link"/>
+        <origin xyz="0.0 0.0 0.12" rpy="0.0 0.0 0.0"/>
+    </joint>
 </robot>
