Commit message: Edit code

File: my_robot_description/urdf/my_robot.gazebo.xacro (robot description, xacro)
@@ -9,4 +9,8 @@
 	    <turnGravityOff>false</turnGravityOff>
     </gazebo>
+    <gazebo reference="uwb_link">
+        <material>Gazebo/White</material>
+        <turnGravityOff>false</turnGravityOff>
+    </gazebo>
     <xacro:macro name="wheel_transmission" params="name">
         <gazebo reference="wheel_${name}_link">
@@ -17,150 +21,150 @@
             <fdir1 value="0.2"/>
             <material>Gazebo/Black</material>
-	        <turnGravityOff>false</turnGravityOff>
+            <turnGravityOff>false</turnGravityOff>
         </gazebo>
         <!-- <transmission name="wheel_${name}_trans">
-  		    <type>transmission_interface/SimpleTransmission</type>
-  		    <actuator name="wheel_${name}_motor">
+            <type>transmission_interface/SimpleTransmission</type>
+            <actuator name="wheel_${name}_motor">
                 <hardwareInterface>hardware_interface/VelocityJointInterface</hardwareInterface>
-			    <mechanicalReduction>1</mechanicalReduction>
-  		    </actuator>
-  		    <joint name="wheel_${name}_joint">
-			    <hardwareInterface>hardware_interface/VelocityJointInterface</hardwareInterface>
-  		    </joint>
+                <mechanicalReduction>1</mechanicalReduction>
+            </actuator>
+            <joint name="wheel_${name}_joint">
+                <hardwareInterface>hardware_interface/VelocityJointInterface</hardwareInterface>
+            </joint>
         </transmission> -->
     </xacro:macro>
-    <xacro:if value="${use_gazebo_simulation}">
-        <!-- <gazebo>
-            <plugin name="differential_drive_controller" filename="libgazebo_ros_diff_drive.so">
-                <alwaysOn>true</alwaysOn>
-                <legacyMode>false</legacyMode>
-                <updateRate>100</updateRate>
-                <leftJoint>wheel_front_left_joint</leftJoint>
-                <rightJoint>wheel_front_right_joint</rightJoint>
-                <wheelSeparation>${wheel_separation}</wheelSeparation>
-                <wheelDiameter>${wheel_radius * 2}</wheelDiameter>
-                <wheelTorque>5</wheelTorque>
-                <torque>5</torque>
-                <commandTopic>/my_robot/cmd_vel</commandTopic>
-                <odometryTopic>odom_gazebo</odometryTopic>
-                <odometryFrame>odom</odometryFrame>
-                <odometrySource >encoder</odometrySource >
-                <publishOdomTF>false</publishOdomTF>
-                <publishWheelTF>false</publishWheelTF>
-                <publishWheelJointState>false</publishWheelJointState>
-                <publishTf>1</publishTf>
-                <robotBaseFrame>base_footprint</robotBaseFrame>
-                <wheelAcceleration>0</wheelAcceleration>
-                <rosDebugLevel>na</rosDebugLevel>
+    <!-- <gazebo>
+        <plugin name="differential_drive_controller" filename="libgazebo_ros_diff_drive.so">
+            <alwaysOn>true</alwaysOn>
+            <legacyMode>false</legacyMode>
+            <updateRate>100</updateRate>
+            <leftJoint>wheel_front_left_joint</leftJoint>
+            <rightJoint>wheel_front_right_joint</rightJoint>
+            <wheelSeparation>${wheel_separation}</wheelSeparation>
+            <wheelDiameter>${wheel_radius * 2}</wheelDiameter>
+            <wheelTorque>5</wheelTorque>
+            <torque>5</torque>
+            <commandTopic>/my_robot/cmd_vel</commandTopic>
+            <odometryTopic>odom_gazebo</odometryTopic>
+            <odometryFrame>odom</odometryFrame>
+            <odometrySource >encoder</odometrySource >
+            <publishOdomTF>false</publishOdomTF>
+            <publishWheelTF>false</publishWheelTF>
+            <publishWheelJointState>false</publishWheelJointState>
+            <publishTf>1</publishTf>
+            <robotBaseFrame>base_footprint</robotBaseFrame>
+            <wheelAcceleration>0</wheelAcceleration>
+            <rosDebugLevel>na</rosDebugLevel>
+        </plugin>
+    </gazebo>
+    <gazebo>
+        <plugin name="differential_drive_controller" filename="libgazebo_ros_diff_drive.so">
+            <alwaysOn>true</alwaysOn>
+            <legacyMode>false</legacyMode>
+            <updateRate>100</updateRate>
+            <leftJoint>wheel_rear_left_joint</leftJoint>
+            <rightJoint>wheel_rear_right_joint</rightJoint>
+            <wheelSeparation>${wheel_separation}</wheelSeparation>
+            <wheelDiameter>${wheel_radius * 2}</wheelDiameter>
+            <wheelTorque>5</wheelTorque>
+            <torque>5</torque>
+            <commandTopic>cmd_vel</commandTopic>
+            <odometryTopic>odom_gazebo</odometryTopic>
+            <odometryFrame>odom</odometryFrame>
+            <odometrySource >encoder</odometrySource >
+            <publishOdomTF>false</publishOdomTF>
+            <publishWheelTF>false</publishWheelTF>
+            <publishWheelJointState>false</publishWheelJointState>
+            <publishTf>1</publishTf>
+            <robotBaseFrame>base_footprint</robotBaseFrame>
+            <wheelAcceleration>0</wheelAcceleration>
+            <rosDebugLevel>na</rosDebugLevel>
+        </plugin>
+    </gazebo> -->
+    <gazebo>
+        <plugin name="skid_steer_drive_controller" filename="libgazebo_ros_skid_steer_drive.so">
+            <alwaysOn>true</alwaysOn>
+            <updateRate>100.0</updateRate>
+            <leftFrontJoint>wheel_front_left_joint</leftFrontJoint>
+            <rightFrontJoint>wheel_front_right_joint</rightFrontJoint>
+            <leftRearJoint>wheel_rear_left_joint</leftRearJoint>
+            <rightRearJoint>wheel_rear_right_joint</rightRearJoint>
+            <wheelSeparation>${wheel_separation}</wheelSeparation>
+            <wheelDiameter>${wheel_radius * 2}</wheelDiameter>
+            <robotBaseFrame>base_link</robotBaseFrame>
+            <torque>5</torque>
+            <commandTopic>cmd_vel</commandTopic>
+            <odometryTopic>odom_gazebo</odometryTopic>
+            <odometryFrame>odom</odometryFrame>
+            <robotBaseFrame>base_footprint</robotBaseFrame>
+            <wheelAcceleration>0</wheelAcceleration>
+            <rosDebugLevel>na</rosDebugLevel>
+            <covariance_x>0.001</covariance_x>
+            <covariance_y>0.001</covariance_y>
+            <covariance_yaw>0.01</covariance_yaw>
+            <broadcastTF>false</broadcastTF>
+        </plugin>
+    </gazebo>
+    <gazebo reference="base_scan">
+        <sensor type="ray" name="lidar">
+            <pose>0 0 0 0 0 0</pose>
+            <visualize>true</visualize>
+            <update_rate>100</update_rate>
+            <ray>
+                <scan>
+                    <horizontal>
+                    <samples>2000</samples>
+                    <resolution>1</resolution>
+                    <min_angle>-${PI}</min_angle>
+                    <max_angle>${PI}</max_angle>
+                    </horizontal>
+                </scan>
+                <range>
+                    <min>0.15</min>
+                    <max>12.0</max>
+                    <resolution>0.01</resolution>
+                </range>
+                <noise>
+                    <type>gaussian</type>
+                    <mean>0.0</mean>
+                    <stddev>0.01</stddev>
+                </noise>
+            </ray>
+            <plugin name="gazebo_ros_head_hokuyo_controller" filename="libgazebo_ros_laser.so">
+                <topicName>/my_robot/scan</topicName>
+                <frameName>base_scan</frameName>
             </plugin>
-        </gazebo>
-        <gazebo>
-            <plugin name="differential_drive_controller" filename="libgazebo_ros_diff_drive.so">
-                <alwaysOn>true</alwaysOn>
-                <legacyMode>false</legacyMode>
-                <updateRate>100</updateRate>
-                <leftJoint>wheel_rear_left_joint</leftJoint>
-                <rightJoint>wheel_rear_right_joint</rightJoint>
-                <wheelSeparation>${wheel_separation}</wheelSeparation>
-                <wheelDiameter>${wheel_radius * 2}</wheelDiameter>
-                <wheelTorque>5</wheelTorque>
-                <torque>5</torque>
-                <commandTopic>cmd_vel</commandTopic>
-                <odometryTopic>odom_gazebo</odometryTopic>
-                <odometryFrame>odom</odometryFrame>
-                <odometrySource >encoder</odometrySource >
-                <publishOdomTF>false</publishOdomTF>
-                <publishWheelTF>false</publishWheelTF>
-                <publishWheelJointState>false</publishWheelJointState>
-                <publishTf>1</publishTf>
-                <robotBaseFrame>base_footprint</robotBaseFrame>
-                <wheelAcceleration>0</wheelAcceleration>
-                <rosDebugLevel>na</rosDebugLevel>
+        </sensor>
+    </gazebo>
+    <gazebo reference="imu_link">
+        <sensor name="imu_sensor" type="imu">
+            <always_on>true</always_on>
+            <update_rate>100</update_rate>
+            <visualize>true</visualize>
+            <topic>/my_robot/imu</topic>
+            <plugin filename="libgazebo_ros_imu_sensor.so" name="imu_plugin">
+                <topicName>/my_robot/imu</topicName>
+                <bodyName>imu_link</bodyName>
+                <updateRateHZ>50.0</updateRateHZ>
+                <gaussianNoise>0.0</gaussianNoise>
+                <xyzOffset>0 0 0</xyzOffset>
+                <rpyOffset>0 0 0</rpyOffset>
+                <frameName>imu_link</frameName>
+                <initialOrientationAsReference>false</initialOrientationAsReference>
             </plugin>
-        </gazebo> -->
-        <gazebo>
-            <plugin name="skid_steer_drive_controller" filename="libgazebo_ros_skid_steer_drive.so">
-                <alwaysOn>true</alwaysOn>
-                <updateRate>100.0</updateRate>
-                <leftFrontJoint>wheel_front_left_joint</leftFrontJoint>
-                <rightFrontJoint>wheel_front_right_joint</rightFrontJoint>
-                <leftRearJoint>wheel_rear_left_joint</leftRearJoint>
-                <rightRearJoint>wheel_rear_right_joint</rightRearJoint>
-                <wheelSeparation>${wheel_separation}</wheelSeparation>
-                <wheelDiameter>${wheel_radius * 2}</wheelDiameter>
-                <robotBaseFrame>base_link</robotBaseFrame>
-                <torque>5</torque>
-                <commandTopic>cmd_vel</commandTopic>
-                <odometryTopic>odom_gazebo</odometryTopic>
-                <odometryFrame>odom</odometryFrame>
-                <robotBaseFrame>base_footprint</robotBaseFrame>
-                <wheelAcceleration>0</wheelAcceleration>
-                <rosDebugLevel>na</rosDebugLevel>
-                <covariance_x>0.001</covariance_x>
-                <covariance_y>0.001</covariance_y>
-                <covariance_yaw>0.01</covariance_yaw>
-                <broadcastTF>false</broadcastTF>
-            </plugin>
-        </gazebo>
-        <gazebo reference="base_scan">
-            <sensor type="ray" name="lidar">
-                <pose>0 0 0 0 0 0</pose>
-                <visualize>true</visualize>
-                <update_rate>50</update_rate>
-                <ray>
-                    <scan>
-                        <horizontal>
-                        <samples>2000</samples>
-                        <resolution>1</resolution>
-                        <min_angle>-${PI}</min_angle>
-                        <max_angle>${PI}</max_angle>
-                        </horizontal>
-                    </scan>
-                    <range>
-                        <min>0.15</min>
-                        <max>12.0</max>
-                        <resolution>0.01</resolution>
-                    </range>
-                    <noise>
-                        <type>gaussian</type>
-                        <mean>0.0</mean>
-                        <stddev>0.01</stddev>
-                    </noise>
-                </ray>
-                <plugin name="gazebo_ros_head_hokuyo_controller" filename="libgazebo_ros_laser.so">
-                    <topicName>/my_robot/scan</topicName>
-                    <frameName>base_scan</frameName>
-                </plugin>
-            </sensor>
-        </gazebo>
-        <gazebo>
-            <plugin name="imu_plugin" filename="libgazebo_ros_imu.so">
-                <alwaysOn>true</alwaysOn>
-                <updateRate>10</updateRate>
-                <bodyName>imu_link</bodyName>
-                <frameName>imu_link</frameName>
-                <topicName>imu</topicName>
-                <serviceName>imu_service</serviceName>
-                <gaussianNoise>0.0</gaussianNoise>
-                <imu>
-                    <noise>
-                        <type>gaussian</type>
-                        <rate>
-                        <mean>0.0</mean>
-                        <stddev>2e-4</stddev>
-                        <bias_mean>0.0000075</bias_mean>
-                        <bias_stddev>0.0000008</bias_stddev>
-                        </rate>
-                        <accel>
-                        <mean>0.0</mean>
-                        <stddev>1.7e-2</stddev>
-                        <bias_mean>0.1</bias_mean>
-                        <bias_stddev>0.001</bias_stddev>
-                        </accel>
-                    </noise>
-                </imu>
-            </plugin>
-        </gazebo>
-    </xacro:if>
+            <pose>0 0 0 0 0 0</pose>
+        </sensor>
+    </gazebo>
+    <gazebo>
+        <plugin name='libgtec_uwb_plugin' filename='libgtec_uwb_plugin.so'>
+            <update_rate>100</update_rate>
+            <nlosSoftWallWidth>0.25</nlosSoftWallWidth>
+            <tag_z_offset>0</tag_z_offset>
+            <tag_link>tag_0</tag_link>
+            <anchor_prefix>uwb_anchor</anchor_prefix>
+            <all_los>false</all_los>
+            <tag_id>0</tag_id>
+        </plugin>
+    </gazebo>
     <gazebo>
         <plugin name="gazebo_ros_control" filename="libgazebo_ros_control.so">

File: my_robot_description/urdf/my_robot.urdf.xacro (robot description, xacro)
@@ -113,3 +113,23 @@
         <origin xyz="0.0 0.0 0.12" rpy="0.0 0.0 0.0"/>
     </joint>
+    <link name="uwb_link">
+        <visual>
+            <origin xyz="0.01125 -0.02425 -0.08" rpy="${PI/2} 0.0 ${PI}"/>
+            <geometry>
+                <mesh filename="package://my_robot_description/meshes/uwb.STL" scale="0.001 0.001 0.001"/>
+            </geometry>
+            <material name="white"/>
+        </visual>
+        <collision>
+            <origin xyz="0.01125 -0.02425 -0.08" rpy="${PI/2} 0.0 ${PI}"/>
+            <geometry>
+                <mesh filename="package://my_robot_description/meshes/uwb.STL" scale="0.001 0.001 0.001"/>
+            </geometry>
+        </collision>
+    </link>
+    <joint name="uwb_joint" type="fixed">
+        <parent link="base_link"/>
+        <child link="uwb_link"/>
+        <origin xyz="0.0 0.0 0.33" rpy="0.0 0.0 0.0"/>
+    </joint>
 </robot>

Commit message: Update code

File: my_robot_description/urdf/my_robot.gazebo.xacro (robot description, xacro)
@@ -3,13 +3,13 @@
     <gazebo reference="base_link">
         <material>Gazebo/SkyBlue</material>
-	    <turnGravityOff>false</turnGravityOff>
+	    <gravity>false</gravity>
     </gazebo>
     <gazebo reference="base_scan">
         <material>Gazebo/Grey</material>
-	    <turnGravityOff>false</turnGravityOff>
+	    <gravity>false</gravity>
     </gazebo>
-    <gazebo reference="uwb_link">
+    <gazebo reference="uwb_tag">
         <material>Gazebo/White</material>
-        <turnGravityOff>false</turnGravityOff>
+        <gravity>false</gravity>
     </gazebo>
     <xacro:macro name="wheel_transmission" params="name">
@@ -21,5 +21,5 @@
             <fdir1 value="0.2"/>
             <material>Gazebo/Black</material>
-            <turnGravityOff>false</turnGravityOff>
+            <gravity>false</gravity>
         </gazebo>
         <!-- <transmission name="wheel_${name}_trans">
@@ -34,5 +34,5 @@
         </transmission> -->
     </xacro:macro>
-    <!-- <gazebo>
+    <gazebo>
         <plugin name="differential_drive_controller" filename="libgazebo_ros_diff_drive.so">
             <alwaysOn>true</alwaysOn>
@@ -81,6 +81,6 @@
             <rosDebugLevel>na</rosDebugLevel>
         </plugin>
-    </gazebo> -->
-    <gazebo>
+    </gazebo>
+    <!-- <gazebo>
         <plugin name="skid_steer_drive_controller" filename="libgazebo_ros_skid_steer_drive.so">
             <alwaysOn>true</alwaysOn>
@@ -105,5 +105,5 @@
             <broadcastTF>false</broadcastTF>
         </plugin>
-    </gazebo>
+    </gazebo> -->
     <gazebo reference="base_scan">
         <sensor type="ray" name="lidar">
@@ -138,11 +138,12 @@
     </gazebo>
     <gazebo reference="imu_link">
+        <gravity>true</gravity>
         <sensor name="imu_sensor" type="imu">
             <always_on>true</always_on>
-            <update_rate>100</update_rate>
+            <update_rate>50</update_rate>
             <visualize>true</visualize>
-            <topic>/my_robot/imu</topic>
+            <topic>imu</topic>
             <plugin filename="libgazebo_ros_imu_sensor.so" name="imu_plugin">
-                <topicName>/my_robot/imu</topicName>
+                <topicName>/my_robot/imu/data_raw</topicName>
                 <bodyName>imu_link</bodyName>
                 <updateRateHZ>50.0</updateRateHZ>
@@ -158,8 +159,8 @@
     <gazebo>
         <plugin name='libgtec_uwb_plugin' filename='libgtec_uwb_plugin.so'>
-            <update_rate>100</update_rate>
+            <update_rate>50</update_rate>
             <nlosSoftWallWidth>0.25</nlosSoftWallWidth>
             <tag_z_offset>0</tag_z_offset>
-            <tag_link>tag_0</tag_link>
+            <tag_link>uwb_tag</tag_link>
             <anchor_prefix>uwb_anchor</anchor_prefix>
             <all_los>false</all_los>

File: my_robot_description/urdf/my_robot.urdf.xacro (robot description, xacro)
@@ -113,5 +113,10 @@
         <origin xyz="0.0 0.0 0.12" rpy="0.0 0.0 0.0"/>
     </joint>
-    <link name="uwb_link">
+    <link name="uwb_tag">
+        <inertial>
+            <origin xyz="0.01125 -0.02425 -0.08" rpy="${PI/2} 0.0 ${PI}"/>
+            <mass value="0.1" />
+            <inertia ixx="0.001" ixy="0.0" ixz="0.0" iyy="0.001" iyz="0.0" izz="0.001" />
+        </inertial>
         <visual>
             <origin xyz="0.01125 -0.02425 -0.08" rpy="${PI/2} 0.0 ${PI}"/>
@@ -128,7 +133,7 @@
         </collision>
     </link>
-    <joint name="uwb_joint" type="fixed">
+    <joint name="uwb_tag_joint" type="fixed">
         <parent link="base_link"/>
-        <child link="uwb_link"/>
+        <child link="uwb_tag"/>
         <origin xyz="0.0 0.0 0.33" rpy="0.0 0.0 0.0"/>
     </joint>
